File: pcb/rear_zone.kicad_sch (KiCad schematic)
At the start: 0 parts

Commit message: Added Front and Rear zone sheets made of CAN and MCU design sheets.
Parts:
- added C25, C27, C28, C29, C30, C33, C34: 100nF, symbol Device:C
- added C26: 470μF, symbol Device:C
- added C31, C32: 1nF, symbol Device:C
- added D10, D16, D17, D18, D6, D7, D8, D9: D_Schottky, symbol Device:D_Schottky
- added J10, J11: Conn_01x06, symbol Connector_Generic:Conn_01x06
- added J20, J21: Conn_01x02, symbol Connector_Generic:Conn_01x02
- added R14, R15, R19: 10kΩ, symbol Device:R_US
- added R16, R17: 20kΩ, symbol Device:R_US
- added R18: 47kΩ, symbol Device:R_US
- added R25, R26: 120Ω, symbol Device:R_Small_US
- added TP22, TP23, TP24, TP25, TP26, TP27, TP40, TP41, TP42, TP43, TP44, TP45, TP46, TP47, TP48, TP49, TP50, TP51, TP52: TestPoint, symbol Connector:TestPoint
- added U7: L298N, Package_TO_SOT_THT:TO-220-15_P2.54x5.08mm_StaggerOdd_Lead4.58mm_Vertical, symbol Driver_Motor:L298N
- added U8, U9: ACS712xLCTR-05B, Package_SO:SOIC-8_3.9x4.9mm_P1.27mm, symbol Sensor_Current:ACS712xLCTR-05B
Connections:
- new net: C31.1, U9.6 (FILTER)
- new net: J21.1 (Pin_1), R26.2
- new net: D17.2 (A), D9.1 (K), U7.13 (OUT3), U9.1 (IP+), U9.2 (IP+)
- new net: D6.1 (K), D7.2 (A), U7.2 (OUT1), U8.1 (IP+), U8.2 (IP+)
- new net: J20.1 (Pin_1), R25.2
- new net: C32.2, U8.6 (FILTER)
- new net +12V: C25.1, C26.1, D16.1 (K), D17.1 (K), D18.1 (K), D7.1 (K), R18.1, U7.4 (Vs)
- new net +3V3: J10.2 (Pin_2), J11.2 (Pin_2)
- new net +5V: C27.2, C33.1, C34.1, U7.9 (Vss), U8.8 (VCC), U9.8 (VCC)
- new net ADC_IN_L: C28.1, R15.2, R16.1
- new net ADC_IN_R: C29.1, R14.2, R17.1
- new net BLINK_L: TP41.1
- new net BLINK_R: TP43.1
- new net CAN_A_H: R26.1
- new net CAN_A_L: J21.2 (Pin_2)
- new net CAN_B_H: R25.1
- new net CAN_B_L: J20.2 (Pin_2)
- new net CAN_RX_A: TP23.1
- new net CAN_RX_B: TP24.1
- new net CAN_TX_A: TP26.1
- new net CAN_TX_B: TP40.1
- new net DEG_A: TP25.1
- new net DEG_B: TP27.1
- new net DIR_A: TP52.1, U7.5 (IN1)
- new net ENC_L_A: J11.3 (Pin_3)
- new net ENC_L_B: J11.4 (Pin_4)
- new net ENC_R_A: J10.3 (Pin_3)
- new net ENC_R_B: J10.4 (Pin_4)
- new net EN_A: TP51.1, U7.6 (EnA)
- new net ERR: TP22.1
- new net GND: C25.2, C26.2, C27.1, C28.2, C29.2, C30.2, C31.2, C32.1, C33.2, C34.2, D10.2 (A), D6.2 (A), D8.2 (A), D9.2 (A), J10.5 (Pin_5), J11.5 (Pin_5), R16.2, R17.2, R19.2, TP45.1, TP47.1, U7.1 (SENSE_A), U7.15 (SENSE_B), U7.8 (GND), U8.5 (GND), U9.5 (GND)
- new net I_L: R15.1, TP46.1, U9.7 (VIOUT)
- new net I_R: R14.1, TP48.1, U8.7 (VIOUT)
- new net MCU/EN_B: U7.11 (EnB)
- new net MCU/IN2: U7.7 (IN2)
- new net MCU/IN3: U7.10 (IN3)
- new net MCU/IN4: U7.12 (IN4)
- new net M_L+: J11.1 (Pin_1), U9.3 (IP-), U9.4 (IP-)
- new net M_L-: D10.1 (K), D18.2 (A), J11.6 (Pin_6), U7.14 (OUT4)
- new net M_R+: J10.1 (Pin_1), U8.3 (IP-), U8.4 (IP-)
- new net M_R-: D16.2 (A), D8.1 (K), J10.6 (Pin_6), U7.3 (OUT2)
- new net OVERLOAD: TP49.1
- new net PWM_SET: TP42.1
- new net TEST_BTN: TP44.1
- new net VBAT: C30.1, R18.2, R19.1, TP50.1
- no-connect marks 0 -> 1
Other:
- added sheet CAN A (can_bus.kicad_sch)
- added sheet CAN B (can_bus.kicad_sch)
- added sheet MCU (STM32F401RE.kicad_sch)
- note added: "Motor Encoder Connectors"
- note added: "Test Points"
- note added: "Voltage Dividers"

Commit message: Added footprints to all components.
Parts:
- C301: renamed from C28; footprint (none) -> Capacitor_SMD:C_0603_1608Metric
- C302: renamed from C29; footprint (none) -> Capacitor_SMD:C_0603_1608Metric
- C303: renamed from C30; footprint (none) -> Capacitor_SMD:C_0603_1608Metric
- C304: renamed from C27; footprint (none) -> Capacitor_SMD:C_0603_1608Metric
- C305: renamed from C26; footprint (none) -> Capacitor_SMD:CP_Elec_8x11.9
- C306: renamed from C25; footprint (none) -> Capacitor_SMD:C_0603_1608Metric
- C307: renamed from C34; footprint (none) -> Capacitor_SMD:C_0603_1608Metric
- C308: renamed from C33; footprint (none) -> Capacitor_SMD:C_0603_1608Metric
- C309: renamed from C32; footprint (none) -> Capacitor_SMD:C_0603_1608Metric
- C310: renamed from C31; footprint (none) -> Capacitor_SMD:C_0603_1608Metric
- D301: renamed from D7; footprint (none) -> Diode_SMD:D_SMB
- D302: renamed from D6; footprint (none) -> Diode_SMD:D_SMB
- D303: renamed from D16; footprint (none) -> Diode_SMD:D_SMB
- D304: renamed from D8; footprint (none) -> Diode_SMD:D_SMB
- D305: renamed from D17; footprint (none) -> Diode_SMD:D_SMB
- D306: renamed from D9; footprint (none) -> Diode_SMD:D_SMB
- D307: renamed from D18; footprint (none) -> Diode_SMD:D_SMB
- D308: renamed from D10; footprint (none) -> Diode_SMD:D_SMB
- J301: renamed from J20; footprint (none) -> Connector_PinHeader_2.54mm:PinHeader_1x02_P2.54mm_Vertical
- J302: renamed from J21; footprint (none) -> Connector_PinHeader_2.54mm:PinHeader_1x02_P2.54mm_Vertical
- J303: renamed from J11; footprint (none) -> Connector_JST:JST_PH_B6B-PH-SM4-TB_1x06-1MP_P2.00mm_Vertical
- J304: renamed from J10; footprint (none) -> Connector_JST:JST_PH_B6B-PH-SM4-TB_1x06-1MP_P2.00mm_Vertical
- R301: renamed from R15; footprint (none) -> Resistor_SMD:R_0603_1608Metric
- R302: renamed from R16; footprint (none) -> Resistor_SMD:R_0603_1608Metric
- R303: renamed from R25; footprint (none) -> Resistor_SMD:R_0603_1608Metric
- R304: renamed from R26; footprint (none) -> Resistor_SMD:R_0603_1608Metric
- R305: renamed from R14; footprint (none) -> Resistor_SMD:R_0603_1608Metric
- R306: renamed from R17; footprint (none) -> Resistor_SMD:R_0603_1608Metric
- R307: renamed from R18; footprint (none) -> Resistor_SMD:R_0603_1608Metric
- R308: renamed from R19; footprint (none) -> Resistor_SMD:R_0603_1608Metric
- TP301: renamed from TP22; footprint (none) -> TestPoint:TestPoint_Keystone_5015_Micro_Mini
- TP302: renamed from TP23; footprint (none) -> TestPoint:TestPoint_Keystone_5015_Micro_Mini
- TP303: renamed from TP24; footprint (none) -> TestPoint:TestPoint_Keystone_5015_Micro_Mini
- TP304: renamed from TP25; footprint (none) -> TestPoint:TestPoint_Keystone_5015_Micro_Mini
- TP305: renamed from TP26; footprint (none) -> TestPoint:TestPoint_Keystone_5015_Micro_Mini
- TP306: renamed from TP27; footprint (none) -> TestPoint:TestPoint_Keystone_5015_Micro_Mini
- TP307: renamed from TP40; footprint (none) -> TestPoint:TestPoint_Keystone_5015_Micro_Mini
- TP308: renamed from TP41; footprint (none) -> TestPoint:TestPoint_Keystone_5015_Micro_Mini
- TP309: renamed from TP42; footprint (none) -> TestPoint:TestPoint_Keystone_5015_Micro_Mini
- TP310: renamed from TP43; footprint (none) -> TestPoint:TestPoint_Keystone_5015_Micro_Mini
- TP311: renamed from TP44; footprint (none) -> TestPoint:TestPoint_Keystone_5015_Micro_Mini
- TP312: renamed from TP45; footprint (none) -> TestPoint:TestPoint_Keystone_5015_Micro_Mini
- TP313: renamed from TP46; footprint (none) -> TestPoint:TestPoint_Keystone_5015_Micro_Mini
- TP314: renamed from TP47; footprint (none) -> TestPoint:TestPoint_Keystone_5015_Micro_Mini
- TP315: renamed from TP49; footprint (none) -> TestPoint:TestPoint_Keystone_5015_Micro_Mini
- TP316: renamed from TP48; footprint (none) -> TestPoint:TestPoint_Keystone_5015_Micro_Mini
- TP317: renamed from TP51; footprint (none) -> TestPoint:TestPoint_Keystone_5015_Micro_Mini
- TP318: renamed from TP50; footprint (none) -> TestPoint:TestPoint_Keystone_5015_Micro_Mini
- TP319: renamed from TP52; footprint (none) -> TestPoint:TestPoint_Keystone_5015_Micro_Mini
- renumbered U7 to U301, U8 to U302, U9 to U303

Commit message: Added CAN Bus connectors and finalized schematic with BOM, LCSC #s, and links to parts.
Parts:
- C301, C302, C303, C304, C307, C308: LCSC (none) -> C18522636; MPN (none) -> KGM15AR71C104KT; Manufacturer (none) -> KYOCERA AVX
- C305: footprint Capacitor_SMD:CP_Elec_8x11.9 -> Capacitor_SMD:CP_Elec_10x12.6; LCSC (none) -> C1517666; MPN (none) -> A768MS477M1ELAE017; Manufacturer (none) -> KEMET
- C306: LCSC (none) -> C14663; MPN (none) -> CC0603KRX7R9BB104; Manufacturer (none) -> YAGEO
- C309, C310: LCSC (none) -> C2219251; MPN (none) -> GCM1885C2A102FA16D; Manufacturer (none) -> Murata
- D301, D302, D303, D304, D305, D306, D307, D308: LCSC (none) -> C139681; MPN (none) -> SK520B; Manufacturer (none) -> SMC Diode Solutions
- J301, J302: LCSC (none) -> C492401; MPN (none) -> PZ254V-11-02P
- J303, J304: LCSC (none) -> C471518; MPN (none) -> B6B-PH-SM4-TB; Manufacturer (none) -> JST
- R301, R305, R308: LCSC (none) -> C844918; MPN (none) -> CRCW060310K0FKEA; Manufacturer (none) -> Vishay Dale
- R302, R306: LCSC (none) -> C4184; MPN (none) -> 0603WAF2002T5E; Manufacturer (none) -> UNI-ROYAL
- R303, R304: LCSC (none) -> C114640; MPN (none) -> RC0603FR-07120RL; Manufacturer (none) -> YAGEO
- R307: LCSC (none) -> C105579; MPN (none) -> RC0603FR-0747KL; Manufacturer (none) -> YAGEO
- TP301, TP302, TP303, TP304, TP305, TP306, TP307, TP308, TP309, TP310, TP311, TP312, TP313, TP314, TP315, TP316, TP317, TP318, TP319: LCSC (none) -> C2906768; MPN (none) -> 5015; Manufacturer (none) -> Keystone Electronics
- U301: LCSC (none) -> C434589; MPN (none) -> L298N; Manufacturer (none) -> STMicroelectronics
- U302, U303: LCSC (none) -> C44471; MPN (none) -> ACS712ELCTR-05B-T; Manufacturer (none) -> Allegro MicroSystems
Other:
- company: (none) -> 18-649 Lab 4: Controller PCB
- title: (none) -> Rear Zone: Drivetrain
