File: pcb/can_bus.kicad_sch (KiCad schematic)
At the start: 13 parts, among them J1 Conn_01x02_Pin, J2 Conn_01x02_Pin, U1 MCP2515-xST, U2 SN65HVD230, Y1 CX3225SB16000H0FLJCC

Commit message: Connected oscillator to controller. Fixed local/hierarchical labeling in sheet.
Connections:
- net +3V3: now also U1.4 (~{TX0RTS}), U1.5 (~{TX1RTS}), U1.7 (~{TX2RTS})
- net CAN_H: no longer J2.1 (Pin_1), U2.7 (CANH)
- net CAN_L: no longer J1.1 (Pin_1), U2.6 (CANL)
- net OSC2: now reaches U1.8 (OSC2)
- net OSC2: now also C2.1, Y1.3
- net OSC1: now reaches U1.9 (OSC1)
- net OSC1: now also C1.1, Y1.1
- new net CAN_H_Local: J2.1 (Pin_1), U2.6 (CANL)
- new net CAN_L_Local: J1.1 (Pin_1), U2.7 (CANH)
Other:
- moved on the sheet: J1, J2, R1

Commit message: Added Front and Rear zone sheets made of CAN and MCU design sheets.
Parts:
- renumbered C4 to C3, C3 to C4, J2 to J1, J1 to J2
Connections:
- net CAN_H_Local: now also U2.7 (CANH); no longer U2.6 (CANL)
- net CAN_L_Local: now also U2.6 (CANL); no longer U2.7 (CANH)

Commit message: Added footprints to all components.
Parts:
- C601: renamed from C1; value 22 pF -> 22pF
- C602: renamed from C2; value 22 pF -> 22pF
- C603: renamed from C3; value 100 nF -> 100nF
- C604: renamed from C4; value 100 nF -> 100nF
- J601: renamed from J1; footprint (none) -> Connector_PinHeader_2.54mm:PinHeader_1x02_P2.54mm_Vertical
- J602: renamed from J2; footprint (none) -> Connector_PinHeader_2.54mm:PinHeader_1x02_P2.54mm_Vertical
- R601: renamed from R1; value 10 kΩ -> 10kΩ
- TP601: renamed from TP1; footprint (none) -> TestPoint:TestPoint_Keystone_5015_Micro_Mini
- TP602: renamed from TP2; footprint (none) -> TestPoint:TestPoint_Keystone_5015_Micro_Mini
- TP603: renamed from TP3; footprint (none) -> TestPoint:TestPoint_Keystone_5015_Micro_Mini
- renumbered U1 to U601, U2 to U602, Y1 to Y601

Commit message: Added CAN Bus connectors and finalized schematic with BOM, LCSC #s, and links to parts.
Parts:
- C601, C602: LCSC (none) -> C2168649; MPN (none) -> C0603C220J1GACTU; Manufacturer (none) -> KEMET
- C603, C604: LCSC (none) -> C18522636; MPN (none) -> KGM15AR71C104KT; Manufacturer (none) -> KYOCERA AVX
- J601, J602: LCSC (none) -> C492401; MPN (none) -> PZ254V-11-02P
- R601: LCSC (none) -> C844918; MPN (none) -> CRCW060310K0FKEA; Manufacturer (none) -> Vishay Dale
- TP601, TP602, TP603: LCSC (none) -> C2906768; MPN (none) -> 5015; Manufacturer (none) -> Keystone Electronics
- U601: LCSC (none) -> C185941; MPN (none) -> MCP2515T-I/ST; Manufacturer (none) -> Microchip Technology
- U602: LCSC (none) -> C2878159; MPN (none) -> SN65HVD230MDREP; Manufacturer (none) -> Texas Instruments
- Y601: LCSC (none) -> C1985207; MPN (none) -> CX3225SB16000H0FLJCC; Manufacturer (none) -> KYOCERA AVX
Other:
- company: (none) -> 18-649 Lab 4: Controller PCB
- title: (none) -> CAN Node: MCP2515 + SN65HVD230 (6 instances)

Commit message: Added final touches and test points.
Parts:
- added TP604, TP605: TestPoint, TestPoint:TestPoint_Keystone_5015_Micro_Mini, symbol Connector:TestPoint
Connections:
- net at U601.1 (TXCAN), U602.1 (D): now also TP605.1
- net at U601.2 (RXCAN), U602.4 (R): now also TP604.1
