File: pcb/front_rear_dual_can.kicad_pcb (KiCad board)
At the start: 2 copper layers, 322 parts, among them J1001 Conn_01x02_Pin, J1002 Conn_01x02_Pin, J101 CAN A Connector, J102 CAN B Connector, J1101 Conn_01x03, J1102 Conn_01x06, J1201 Conn_01x02_Pin, J1202 Conn_01x02_Pin, J1301 Conn_01x02_Pin, J1302 Conn_01x02_Pin, J201 Conn_01x02, J202 Conn_01x02, J203 Conn_01x03, J301 Conn_01x02, J302 Conn_01x02, J303 Conn_01x06, J304 Conn_01x06, J401 Raspberry_Pi_4, J501 XT60, J502 Conn_01x02, J503 Conn_01x02, J504 Conn_01x02, J505 Conn_01x02, J506 Conn_01x02, J601 Conn_01x02_Pin, J602 Conn_01x02_Pin, J701 Conn_01x03, J702 Conn_01x06, J801 Conn_01x02_Pin, J802 Conn_01x02_Pin, J901 Conn_01x02_Pin, J902 Conn_01x02_Pin, Q501 IPD90P03P4L-04-HXY, U1001 MCP2515-xST, U1002 SN65HVD230, U1101 STM32F401RETx, U1201 MCP2515-xST, U1202 SN65HVD230, U1301 MCP2515-xST, U1302 SN65HVD230, U201 INA180A1, U301 L298N, U302 ACS712xLCTR-05B, U303 ACS712xLCTR-05B, U501 TPS564252DRLR, U502 TPS564252DRLR, U503 TPS564252DRLR, U601 MCP2515-xST, U602 SN65HVD230, U701 STM32F401RETx, U801 MCP2515-xST, U802 SN65HVD230, U901 MCP2515-xST, U902 SN65HVD230, Y1001 CX3225SB16000H0FLJCC, Y1101 CX3225SB16000H0FLJCC, Y1201 CX3225SB16000H0FLJCC, Y1301 CX3225SB16000H0FLJCC, Y601 CX3225SB16000H0FLJCC, Y701 CX3225SB16000H0FLJCC, Y801 CX3225SB16000H0FLJCC, Y901 CX3225SB16000H0FLJCC

Commit message: more progress with layout
Parts:
- moved C801 170.0 mm to (239.7, 71.4)
- moved C802 170.0 mm to (239.7, 73.9)
- moved C803 170.0 mm to (239.7, 76.5)
- moved C804 170.0 mm to (239.7, 79.0)
- moved J801 170.0 mm to (244.0, 72.5)
- moved J802 170.0 mm to (248.6, 72.5)
- moved R801 170.0 mm to (239.7, 81.5)
- moved TP801 170.0 mm to (235.0, 64.0)
- moved TP802 170.0 mm to (235.0, 67.8)
- moved TP803 170.0 mm to (235.0, 71.5)
- moved TP804 170.0 mm to (235.0, 75.2)
- moved TP805 170.0 mm to (235.0, 79.0)
- moved U801 170.0 mm to (242.4, 66.2)
- moved U802 170.0 mm to (245.9, 80.7)
- moved C601 151.2 mm to (240.2, 39.9)
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
Commit message: more layout work
Parts:
- added REF**: MountingHole_3.2mm_M3_Pad_Via, MountingHole:MountingHole_3.2mm_M3_Pad_Via, F.Cu at (78.0, 54.2)
- added REF**: MountingHole_3.2mm_M3_Pad_Via, MountingHole:MountingHole_3.2mm_M3_Pad_Via, F.Cu at (78.0, 151.8)
- added REF**: MountingHole_3.2mm_M3_Pad_Via, MountingHole:MountingHole_3.2mm_M3_Pad_Via, F.Cu at (4.99, 102.8)
- added REF**: MountingHole_3.2mm_M3_Pad_Via, MountingHole:MountingHole_3.2mm_M3_Pad_Via, F.Cu at (78.0, 5.17)
- added REF**: MountingHole_3.2mm_M3_Pad_Via, MountingHole:MountingHole_3.2mm_M3_Pad_Via, F.Cu at (4.99, 151.8)
- added REF**: MountingHole_3.2mm_M3_Pad_Via, MountingHole:MountingHole_3.2mm_M3_Pad_Via, F.Cu at (4.99, 54.2)
- added REF**: MountingHole_3.2mm_M3_Pad_Via, MountingHole:MountingHole_3.2mm_M3_Pad_Via, F.Cu at (78.0, 102.8)
- added REF**: MountingHole_3.2mm_M3_Pad_Via, MountingHole:MountingHole_3.2mm_M3_Pad_Via, F.Cu at (4.99, 5.17)
- moved C1001 289.1 mm to (-42.2, 174.0)
- moved C1002 289.1 mm to (-42.2, 176.5)
- moved C1003 289.1 mm to (-42.2, 179.0)
- moved C1004 289.1 mm to (-42.2, 181.5)
- moved C901 289.1 mm to (-62.8, 174.0)
- moved C902 289.1 mm to (-62.8, 176.5)
- moved C903 289.1 mm to (-62.8, 179.0)
- moved C904 289.1 mm to (-62.8, 181.5)
- moved J1001 289.1 mm to (-37.9, 175.0)
- moved J1002 289.1 mm to (-33.3, 175.0)
- moved J901 289.1 mm to (-58.5, 175.0)
- moved J902 289.1 mm to (-53.9, 175.0)
- moved R1001 289.1 mm to (-42.2, 184.0)
- moved R901 289.1 mm to (-62.8, 184.0)
- moved TP1001 289.1 mm to (-46.9, 166.6)
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Routing:
- net GND: track 0.00 -> 77.8 mm, vias 0 -> 45
- net /Rear Zone/MCU/RST: track 0.00 -> 55.7 mm, vias 0 -> 4
- net +3V3: track 0.00 -> 49.5 mm, vias 0 -> 2
- net /Rear Zone/TEST_BTN: track 0.00 -> 22.6 mm
- net /Rear Zone/MCU/SWDIO: track 0.00 -> 21.5 mm
- net /Front Zone/MCU/RST: track 0.00 -> 21.0 mm
- net /Rear Zone/MCU/SWCLK: track 0.00 -> 19.1 mm
- net /Front Zone/TEST_BTN: track 0.00 -> 19.1 mm
- net /Rear Zone/DEG_B: track 0.00 -> 18.3 mm, vias 0 -> 2
- net /Rear Zone/BLINK_R: track 0.00 -> 17.6 mm, vias 0 -> 2
- net /Front Zone/ERR: track 0.00 -> 16.3 mm
- net /Rear Zone/ERR: track 0.00 -> 14.3 mm, vias 0 -> 2
- net /Rear Zone/MCU/OSC_IN: track 0.00 -> 14.0 mm
- net /Front Zone/BLINK_L: track 0.00 -> 13.6 mm
- net /Front Zone/DEG_B: track 0.00 -> 11.9 mm, vias 0 -> 2
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- added copper zone on F.Cu, net GND
- added copper zone on In1.Cu, net GND
Other:
- board outline added: 83 x 157 mm
- copper layers 2 -> 4
- board text added: "BLINK_L"
- board text added: "BLINK_R"
- board text added: "DEBUG"
- board text added: "DEG_A"
- board text added: "DEG_B"
- board text added: "ERR"
- board text added: "RESET"
- board text added: "TEST"

Commit message: holy shit this is taking an eternity
Parts:
- TP1001, TP1002, TP1003, TP1004, TP1005, TP1201, TP1202, TP1203, TP1204, TP1205, TP1301, TP1302, TP1303, TP1304, TP1305, TP201, TP202, TP203, TP204, TP205, TP206, TP207, TP208, TP209, TP210, TP211, TP212, TP213, TP214, TP215, TP301, TP302, TP303, TP304, TP305, TP306, TP307, TP308, TP309, TP310, TP311, TP312, TP313, TP314, TP315, TP316, TP317, TP318, TP319, TP401, TP402, TP403, TP404, TP405, TP406, TP407, TP408, TP409, TP410, TP501, TP502, TP503, TP504, TP505, TP506, TP507, TP508, TP509, TP510, TP601, TP602, TP603, TP604, TP605, TP801, TP802, TP803, TP804, TP805, TP901, TP902, TP903, TP904, TP905: footprint TestPoint:TestPoint_Keystone_5015_Micro_Mini -> TestPoint:TestPoint_Pad_D1.5mm
- moved U1202 321.7 mm to (164.2, 54.1), turned to 90 degrees
- moved U1201 304.2 mm to (163.8, 64.4), turned to -90 degrees
- moved C1201 295.8 mm to (101.7, 39.5)
- moved C1202 295.8 mm to (101.7, 42.1)
- moved C1203 295.8 mm to (101.7, 44.6)
- moved C1204 295.8 mm to (101.7, 47.1)
- moved J1201 295.8 mm to (106.0, 40.6)
- moved J1202 295.8 mm to (110.6, 40.6)
- moved TP1201 295.8 mm to (97.0, 32.1)
- moved TP1202 295.8 mm to (97.0, 35.9)
- moved TP1203 295.8 mm to (97.0, 39.6)
- moved TP1204 295.8 mm to (97.0, 43.4)
- moved TP1205 295.8 mm to (97.0, 47.1)
- moved C1301 275.1 mm to (144.7, 41.8)
- moved C1302 275.1 mm to (144.7, 44.3)
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Routing:
- net +3V3: track 49.5 -> 187.5 mm, vias 2 -> 12
- net GND: track 77.8 -> 136.0 mm, vias 45 -> 76
- net /Front Zone/CAN A/SI: track 0.00 -> 46.5 mm, vias 0 -> 7
- net /Rear Zone/CAN A/SO: track 0.00 -> 42.2 mm, vias 0 -> 4
- net /Front Zone/CAN A/SCK: track 0.00 -> 41.5 mm, vias 0 -> 5
- net /Rear Zone/CAN A/SCK: track 0.00 -> 41.3 mm, vias 0 -> 4
- net /Rear Zone/CAN A/SI: track 0.00 -> 40.2 mm, vias 0 -> 4
- net /Front Zone/CAN A/SO: track 0.00 -> 40.1 mm, vias 0 -> 6
- net /Front Zone/CAN B/CS: track 0.00 -> 38.3 mm, vias 0 -> 7
- net /Front Zone/MCU/RST: track 21.0 -> 54.2 mm, vias 0 -> 2
- net /Rear Zone/CAN A/INT: track 0.00 -> 30.4 mm, vias 0 -> 4
- net /Rear Zone/CAN A/CS: track 0.00 -> 22.2 mm, vias 0 -> 2
- net /Front Zone/CAN B/INT: track 0.00 -> 20.3 mm, vias 0 -> 2
- net /Front Zone/MCU/SWDIO: track 0.00 -> 19.6 mm, vias 0 -> 2
- net /Front Zone/MCU/SWCLK: track 0.00 -> 19.6 mm, vias 0 -> 2
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
Commit message: more progress
Parts:
- moved TP208 274.9 mm to (99.2, -29.0)
- moved TP214 274.9 mm to (104.6, -29.0)
- moved TP215 274.9 mm to (104.6, -25.2)
- moved TP402 274.9 mm to (81.2, -29.0)
- moved TP403 274.9 mm to (81.2, -25.2)
- moved TP404 274.9 mm to (81.2, -21.5)
- moved TP405 274.9 mm to (81.2, -17.8)
- moved TP407 274.9 mm to (86.5, -29.0)
- moved TP408 274.9 mm to (86.5, -25.2)
- moved TP409 274.9 mm to (86.5, -21.5)
- moved J202 274.3 mm to (166.8, 26.0), turned to 180 degrees
- moved TP206 272.8 mm to (149.8, 32.0)
- moved R201 272.1 mm to (101.3, -17.8)
- moved R202 272.1 mm to (101.3, -15.2)
- moved U201 271.9 mm to (109.4, -2.00)
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Routing:
- net GND: track 136.0 -> 205.7 mm, vias 76 -> 101
- net +3V3: track 187.5 -> 244.7 mm, vias 12 -> 14
- net /Front Zone/MCU/ADC1_12: track 0.00 -> 26.7 mm, vias 0 -> 2
- net /Front Zone/MCU/RST: track 54.2 -> 27.9 mm
- net /Cockpit/CAN A/CAN_H_Local: track 0.00 -> 23.7 mm
- net /Front Zone/CAN_TX_A: track 0.00 -> 22.7 mm, vias 0 -> 2
- net /Cockpit/TEST_BTN: track 0.00 -> 22.4 mm
- net Net-(U1201-TXCAN): track 0.00 -> 20.7 mm, vias 0 -> 2
- net /Cockpit/CAN A/SCK: track 0.00 -> 17.1 mm, vias 0 -> 2
- net /Front Zone/CAN_RX_B: track 0.00 -> 17.0 mm, vias 0 -> 2
- net /Cockpit/CAN A/SI: track 0.00 -> 16.6 mm, vias 0 -> 3
- net /Cockpit/CAN B/OSC1: track 0.00 -> 16.2 mm, vias 0 -> 2
- net /Cockpit/CAN A/SO: track 0.00 -> 15.6 mm, vias 0 -> 4
- net /Cockpit/CAN A/INT: track 0.00 -> 15.5 mm
- net Net-(U1201-RXCAN): track 0.00 -> 14.7 mm, vias 0 -> 2
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
Commit message: more work lol
Parts:
- moved R1201 276.3 mm to (39.2, 8.82), turned to 90 degrees
- moved Y601 264.3 mm to (157.8, -1.35)
- moved Y801 226.4 mm to (94.1, 19.1)
- moved Y901 153.0 mm to (165.2, 149.4), turned to 90 degrees
- moved U302 125.6 mm to (48.4, 264.3)
- moved U303 125.6 mm to (48.4, 270.9)
- moved Y1001 110.1 mm to (110.1, 155.8), turned to 90 degrees
- moved TP1003 90.7 mm to (95.8, 146.0)
- moved C1105 89.3 mm to (141.3, 135.6)
- moved C901 89.3 mm to (156.8, 138.7)
- moved C902 89.3 mm to (156.8, 140.2)
- moved C903 89.3 mm to (156.8, 141.7)
- moved C904 89.3 mm to (156.8, 143.2)
- moved S1101 89.3 mm to (149.8, 132.8)
- moved TP904 89.3 mm to (163.6, 138.2)
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Routing:
- net GND: track 205.7 -> 171.4 mm, vias 101 -> 66
- net /Front Zone/CAN_TX_A: track 22.7 -> 0.00 mm, vias 2 -> 0
- net /Front Zone/CAN_RX_B: track 17.0 -> 0.00 mm, vias 2 -> 0
- net /Front Zone/SRV: track 8.78 -> 0.00 mm, vias 2 -> 0
- net /Front Zone/RELAY: track 7.72 -> 0.00 mm, vias 2 -> 0
- net /Front Zone/DEG_A: track 10.3 -> 2.83 mm, vias 2 -> 0
- net /Cockpit/CAN B/OSC2: track 14.1 -> 6.77 mm, vias 2 -> 0
- net /Cockpit/CAN B/OSC1: track 16.2 -> 8.88 mm, vias 2 -> 0
- net /Cockpit/CAN B/CS: track 7.01 -> 0.00 mm
- net /Rear Zone/CAN B/OSC1: track 2.14 -> 8.12 mm, vias 0 -> 2
- net Net-(U1201-~{RESET}): track 0.00 -> 5.97 mm
- net +3V3: track 244.7 -> 239.3 mm, vias 14 -> 12
- net /Front Zone/DEG_B: track 17.1 -> 11.9 mm, vias 4 -> 2
- net /Front Zone/ERR: track 20.5 -> 16.3 mm, vias 2 -> 0
- net /Front Zone/MCU/RST: track 27.9 -> 23.9 mm, vias 2 -> 0
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